File: pcb_proj.kicad_pcb (KiCad board)
At the start: 2 copper layers, 662 parts, among them J1 Conn_02x32_Top_Bottom, J2 Conn_02x10_Top_Bottom, U0 OPA333xxDBV, U1 OPA333xxDBV, U2 OPA333xxDBV, U3 OPA333xxDBV, U4 OPA333xxDBV, U5 OPA333xxDBV, U6 OPA333xxDBV, U7 OPA333xxDBV, U8 OPA333xxDBV, U9 OPA333xxDBV

Commit message: Circuit complete
Committing before I read in netlist just in case things get screwed
Parts:
- moved R6 227.8 mm to (-97.8, 128.3)
- moved U0 227.8 mm to (-53.3, 130.8)
- moved U1 227.8 mm to (-43.2, 128.3)
- moved U2 227.8 mm to (-31.8, 130.8)
- moved U5 227.8 mm to (-1.27, 130.8)
- moved U8 227.8 mm to (24.1, 128.3)
- moved U9 227.8 mm to (-11.4, 135.9)
- moved R0 227.8 mm to (-77.5, 135.9)
- moved R1 227.8 mm to (-81.3, 138.4)
- moved R2 227.8 mm to (-86.4, 134.6)
- moved R3 227.8 mm to (-94.0, 133.3)
- moved R4 227.8 mm to (-104.1, 130.8)
- moved R5 227.8 mm to (-113.0, 132.1)
- moved R7 227.8 mm to (-81.3, 129.5)
- moved R8 227.8 mm to (-94.0, 139.7)
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
Commit message: Additional wires on PCB
Parts:
- added R01: 1k, Resistors_SMD:R_1206, F.Cu at (67.3, 134.6)
- added R02: 1k, Resistors_SMD:R_1206, F.Cu at (78.7, 134.6)
- added R10, R11, R20, R21, R30, R31, R40, R41, R50, R51, R60, R61, R70, R71, R80, R81, R90, R91: 1k, Resistors_SMD:R_1206, F.Cu at (40.6, 132.1)
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Connections:
- R0 pad 1: /op_amps/out0_v -> Net-(R0-Pad1)
- R1 pad 1: /op_amps/out1_v -> Net-(R1-Pad1)
- R16_0 pad 1: /resistor_network/inputs 16-31/out0_i -> /resistor_network/OUT0
- R16_0 pad 2: /resistor_network/inputs 16-31/in16_v -> /C16
- R16_1 pad 1: /resistor_network/inputs 16-31/out1_i -> /resistor_network/OUT1
- R16_1 pad 2: /resistor_network/inputs 16-31/in16_v -> /C16
- R16_2 pad 1: /resistor_network/inputs 16-31/out2_i -> /resistor_network/OUT2
- R16_2 pad 2: /resistor_network/inputs 16-31/in16_v -> /C16
- R16_3 pad 1: /resistor_network/inputs 16-31/out3_i -> /resistor_network/OUT3
- R16_3 pad 2: /resistor_network/inputs 16-31/in16_v -> /C16
- R16_4 pad 1: /resistor_network/inputs 16-31/out4_i -> /resistor_network/OUT4
- R16_4 pad 2: /resistor_network/inputs 16-31/in16_v -> /C16
- R16_5 pad 1: /resistor_network/inputs 16-31/out5_i -> /resistor_network/OUT5
- R16_5 pad 2: /resistor_network/inputs 16-31/in16_v -> /C16
- R16_6 pad 1: /resistor_network/inputs 16-31/out6_i -> /resistor_network/OUT6
- R16_6 pad 2: /resistor_network/inputs 16-31/in16_v -> /C16
- R16_7 pad 1: /resistor_network/inputs 16-31/out7_i -> /resistor_network/OUT7
- R16_7 pad 2: /resistor_network/inputs 16-31/in16_v -> /C16
- R16_8 pad 1: /resistor_network/inputs 16-31/out8_i -> /resistor_network/OUT8
- R16_8 pad 2: /resistor_network/inputs 16-31/in16_v -> /C16
- R16_9 pad 1: /resistor_network/inputs 16-31/out9_i -> /resistor_network/OUT9
- R16_9 pad 2: /resistor_network/inputs 16-31/in16_v -> /C16
- R17_0 pad 1: /resistor_network/inputs 16-31/out0_i -> /resistor_network/OUT0
- R17_0 pad 2: /resistor_network/inputs 16-31/in17_v -> /C17
- R17_1 pad 1: /resistor_network/inputs 16-31/out1_i -> /resistor_network/OUT1
- R17_1 pad 2: /resistor_network/inputs 16-31/in17_v -> /C17
- R17_2 pad 1: /resistor_network/inputs 16-31/out2_i -> /resistor_network/OUT2
- R17_2 pad 2: /resistor_network/inputs 16-31/in17_v -> /C17
- R17_3 pad 1: /resistor_network/inputs 16-31/out3_i -> /resistor_network/OUT3
- R17_3 pad 2: /resistor_network/inputs 16-31/in17_v -> /C17
- R17_4 pad 1: /resistor_network/inputs 16-31/out4_i -> /resistor_network/OUT4
- R17_4 pad 2: /resistor_network/inputs 16-31/in17_v -> /C17
- R17_5 pad 1: /resistor_network/inputs 16-31/out5_i -> /resistor_network/OUT5
- R17_5 pad 2: /resistor_network/inputs 16-31/in17_v -> /C17
- R17_6 pad 1: /resistor_network/inputs 16-31/out6_i -> /resistor_network/OUT6
- R17_6 pad 2: /resistor_network/inputs 16-31/in17_v -> /C17
- R17_7 pad 1: /resistor_network/inputs 16-31/out7_i -> /resistor_network/OUT7
- R17_7 pad 2: /resistor_network/inputs 16-31/in17_v -> /C17
- R17_8 pad 1: /resistor_network/inputs 16-31/out8_i -> /resistor_network/OUT8
- R17_8 pad 2: /resistor_network/inputs 16-31/in17_v -> /C17
- R17_9 pad 1: /resistor_network/inputs 16-31/out9_i -> /resistor_network/OUT9
- R17_9 pad 2: /resistor_network/inputs 16-31/in17_v -> /C17
- R18_0 pad 1: /resistor_network/inputs 16-31/out0_i -> /resistor_network/OUT0
- R18_0 pad 2: /resistor_network/inputs 16-31/in18_v -> /C18
- R18_1 pad 1: /resistor_network/inputs 16-31/out1_i -> /resistor_network/OUT1
- R18_1 pad 2: /resistor_network/inputs 16-31/in18_v -> /C18
- R18_2 pad 1: /resistor_network/inputs 16-31/out2_i -> /resistor_network/OUT2
- R18_2 pad 2: /resistor_network/inputs 16-31/in18_v -> /C18
- R18_3 pad 1: /resistor_network/inputs 16-31/out3_i -> /resistor_network/OUT3
- R18_3 pad 2: /resistor_network/inputs 16-31/in18_v -> /C18
- R18_4 pad 1: /resistor_network/inputs 16-31/out4_i -> /resistor_network/OUT4
- R18_4 pad 2: /resistor_network/inputs 16-31/in18_v -> /C18
- R18_5 pad 1: /resistor_network/inputs 16-31/out5_i -> /resistor_network/OUT5
- R18_5 pad 2: /resistor_network/inputs 16-31/in18_v -> /C18
- R18_6 pad 1: /resistor_network/inputs 16-31/out6_i -> /resistor_network/OUT6
- R18_6 pad 2: /resistor_network/inputs 16-31/in18_v -> /C18
- R18_7 pad 1: /resistor_network/inputs 16-31/out7_i -> /resistor_network/OUT7
- R18_7 pad 2: /resistor_network/inputs 16-31/in18_v -> /C18
- R18_8 pad 1: /resistor_network/inputs 16-31/out8_i -> /resistor_network/OUT8
- R18_8 pad 2: /resistor_network/inputs 16-31/in18_v -> /C18
- R18_9 pad 1: /resistor_network/inputs 16-31/out9_i -> /resistor_network/OUT9
- R18_9 pad 2: /resistor_network/inputs 16-31/in18_v -> /C18
- R19_0 pad 1: /resistor_network/inputs 16-31/out0_i -> /resistor_network/OUT0
- R19_0 pad 2: /resistor_network/inputs 16-31/in19_v -> /C19
- R19_1 pad 1: /resistor_network/inputs 16-31/out1_i -> /resistor_network/OUT1
- R19_1 pad 2: /resistor_network/inputs 16-31/in19_v -> /C19
- R19_2 pad 1: /resistor_network/inputs 16-31/out2_i -> /resistor_network/OUT2
- R19_2 pad 2: /resistor_network/inputs 16-31/in19_v -> /C19
- R19_3 pad 1: /resistor_network/inputs 16-31/out3_i -> /resistor_network/OUT3
- R19_3 pad 2: /resistor_network/inputs 16-31/in19_v -> /C19
- R19_4 pad 1: /resistor_network/inputs 16-31/out4_i -> /resistor_network/OUT4
- R19_4 pad 2: /resistor_network/inputs 16-31/in19_v -> /C19
- R19_5 pad 1: /resistor_network/inputs 16-31/out5_i -> /resistor_network/OUT5
- R19_5 pad 2: /resistor_network/inputs 16-31/in19_v -> /C19
- R19_6 pad 1: /resistor_network/inputs 16-31/out6_i -> /resistor_network/OUT6
- R19_6 pad 2: /resistor_network/inputs 16-31/in19_v -> /C19
- R19_7 pad 1: /resistor_network/inputs 16-31/out7_i -> /resistor_network/OUT7
- R19_7 pad 2: /resistor_network/inputs 16-31/in19_v -> /C19
- R19_8 pad 1: /resistor_network/inputs 16-31/out8_i -> /resistor_network/OUT8
- R19_8 pad 2: /resistor_network/inputs 16-31/in19_v -> /C19
- R19_9 pad 1: /resistor_network/inputs 16-31/out9_i -> /resistor_network/OUT9
- R19_9 pad 2: /resistor_network/inputs 16-31/in19_v -> /C19
- R2 pad 1: /op_amps/out2_v -> Net-(R2-Pad1)
- R20_0 pad 1: /resistor_network/inputs 16-31/out0_i -> /resistor_network/OUT0
- R20_0 pad 2: /resistor_network/inputs 16-31/in20_v -> /C20
- R20_1 pad 1: /resistor_network/inputs 16-31/out1_i -> /resistor_network/OUT1
- R20_1 pad 2: /resistor_network/inputs 16-31/in20_v -> /C20
- R20_2 pad 1: /resistor_network/inputs 16-31/out2_i -> /resistor_network/OUT2
- R20_2 pad 2: /resistor_network/inputs 16-31/in20_v -> /C20
- R20_3 pad 1: /resistor_network/inputs 16-31/out3_i -> /resistor_network/OUT3
- R20_3 pad 2: /resistor_network/inputs 16-31/in20_v -> /C20
- R20_4 pad 1: /resistor_network/inputs 16-31/out4_i -> /resistor_network/OUT4
- R20_4 pad 2: /resistor_network/inputs 16-31/in20_v -> /C20
- R20_5 pad 1: /resistor_network/inputs 16-31/out5_i -> /resistor_network/OUT5
- R20_5 pad 2: /resistor_network/inputs 16-31/in20_v -> /C20
- R20_6 pad 1: /resistor_network/inputs 16-31/out6_i -> /resistor_network/OUT6
- R20_6 pad 2: /resistor_network/inputs 16-31/in20_v -> /C20
- R20_7 pad 1: /resistor_network/inputs 16-31/out7_i -> /resistor_network/OUT7
- R20_7 pad 2: /resistor_network/inputs 16-31/in20_v -> /C20
- R20_8 pad 1: /resistor_network/inputs 16-31/out8_i -> /resistor_network/OUT8
- R20_8 pad 2: /resistor_network/inputs 16-31/in20_v -> /C20
- R20_9 pad 1: /resistor_network/inputs 16-31/out9_i -> /resistor_network/OUT9
- R20_9 pad 2: /resistor_network/inputs 16-31/in20_v -> /C20
- R21_0 pad 1: /resistor_network/inputs 16-31/out0_i -> /resistor_network/OUT0
- R21_0 pad 2: /resistor_network/inputs 16-31/in21_v -> /C21
- R21_1 pad 1: /resistor_network/inputs 16-31/out1_i -> /resistor_network/OUT1
- R21_1 pad 2: /resistor_network/inputs 16-31/in21_v -> /C21
- R21_2 pad 1: /resistor_network/inputs 16-31/out2_i -> /resistor_network/OUT2
- R21_2 pad 2: /resistor_network/inputs 16-31/in21_v -> /C21
- R21_3 pad 1: /resistor_network/inputs 16-31/out3_i -> /resistor_network/OUT3
- R21_3 pad 2: /resistor_network/inputs 16-31/in21_v -> /C21
- R21_4 pad 1: /resistor_network/inputs 16-31/out4_i -> /resistor_network/OUT4
- R21_4 pad 2: /resistor_network/inputs 16-31/in21_v -> /C21
- R21_5 pad 1: /resistor_network/inputs 16-31/out5_i -> /resistor_network/OUT5
- R21_5 pad 2: /resistor_network/inputs 16-31/in21_v -> /C21
- R21_6 pad 1: /resistor_network/inputs 16-31/out6_i -> /resistor_network/OUT6
- R21_6 pad 2: /resistor_network/inputs 16-31/in21_v -> /C21
- R21_7 pad 1: /resistor_network/inputs 16-31/out7_i -> /resistor_network/OUT7
- R21_7 pad 2: /resistor_network/inputs 16-31/in21_v -> /C21
- R21_8 pad 1: /resistor_network/inputs 16-31/out8_i -> /resistor_network/OUT8
- R21_8 pad 2: /resistor_network/inputs 16-31/in21_v -> /C21
- R21_9 pad 1: /resistor_network/inputs 16-31/out9_i -> /resistor_network/OUT9
- R21_9 pad 2: /resistor_network/inputs 16-31/in21_v -> /C21
- R22_0 pad 1: /resistor_network/inputs 16-31/out0_i -> /resistor_network/OUT0
- R22_0 pad 2: /resistor_network/inputs 16-31/in22_v -> /C22
- R22_1 pad 1: /resistor_network/inputs 16-31/out1_i -> /resistor_network/OUT1
- R22_1 pad 2: /resistor_network/inputs 16-31/in22_v -> /C22
- R22_2 pad 1: /resistor_network/inputs 16-31/out2_i -> /resistor_network/OUT2
- R22_2 pad 2: /resistor_network/inputs 16-31/in22_v -> /C22
- R22_3 pad 1: /resistor_network/inputs 16-31/out3_i -> /resistor_network/OUT3
- R22_3 pad 2: /resistor_network/inputs 16-31/in22_v -> /C22
- R22_4 pad 1: /resistor_network/inputs 16-31/out4_i -> /resistor_network/OUT4
- R22_4 pad 2: /resistor_network/inputs 16-31/in22_v -> /C22
- R22_5 pad 1: /resistor_network/inputs 16-31/out5_i -> /resistor_network/OUT5
- R22_5 pad 2: /resistor_network/inputs 16-31/in22_v -> /C22
- R22_6 pad 1: /resistor_network/inputs 16-31/out6_i -> /resistor_network/OUT6
- R22_6 pad 2: /resistor_network/inputs 16-31/in22_v -> /C22
- R22_7 pad 1: /resistor_network/inputs 16-31/out7_i -> /resistor_network/OUT7
- R22_7 pad 2: /resistor_network/inputs 16-31/in22_v -> /C22
- R22_8 pad 1: /resistor_network/inputs 16-31/out8_i -> /resistor_network/OUT8
- R22_8 pad 2: /resistor_network/inputs 16-31/in22_v -> /C22
- R22_9 pad 1: /resistor_network/inputs 16-31/out9_i -> /resistor_network/OUT9
- R22_9 pad 2: /resistor_network/inputs 16-31/in22_v -> /C22
- R23_0 pad 1: /resistor_network/inputs 16-31/out0_i -> /resistor_network/OUT0
- R23_0 pad 2: /resistor_network/inputs 16-31/in23_v -> /C23
- R23_1 pad 1: /resistor_network/inputs 16-31/out1_i -> /resistor_network/OUT1
- R23_1 pad 2: /resistor_network/inputs 16-31/in23_v -> /C23
- R23_2 pad 1: /resistor_network/inputs 16-31/out2_i -> /resistor_network/OUT2
- R23_2 pad 2: /resistor_network/inputs 16-31/in23_v -> /C23
- R23_3 pad 1: /resistor_network/inputs 16-31/out3_i -> /resistor_network/OUT3
- R23_3 pad 2: /resistor_network/inputs 16-31/in23_v -> /C23
- R23_4 pad 1: /resistor_network/inputs 16-31/out4_i -> /resistor_network/OUT4
- R23_4 pad 2: /resistor_network/inputs 16-31/in23_v -> /C23
- R23_5 pad 1: /resistor_network/inputs 16-31/out5_i -> /resistor_network/OUT5
- R23_5 pad 2: /resistor_network/inputs 16-31/in23_v -> /C23
- R23_6 pad 1: /resistor_network/inputs 16-31/out6_i -> /resistor_network/OUT6
- R23_6 pad 2: /resistor_network/inputs 16-31/in23_v -> /C23
- R23_7 pad 1: /resistor_network/inputs 16-31/out7_i -> /resistor_network/OUT7
- R23_7 pad 2: /resistor_network/inputs 16-31/in23_v -> /C23
- R23_8 pad 1: /resistor_network/inputs 16-31/out8_i -> /resistor_network/OUT8
- R23_8 pad 2: /resistor_network/inputs 16-31/in23_v -> /C23
- R23_9 pad 1: /resistor_network/inputs 16-31/out9_i -> /resistor_network/OUT9
- R23_9 pad 2: /resistor_network/inputs 16-31/in23_v -> /C23
- R24_0 pad 1: /resistor_network/inputs 16-31/out0_i -> /resistor_network/OUT0
- R24_0 pad 2: /resistor_network/inputs 16-31/in24_v -> /C24
- R24_1 pad 1: /resistor_network/inputs 16-31/out1_i -> /resistor_network/OUT1
- R24_1 pad 2: /resistor_network/inputs 16-31/in24_v -> /C24
- R24_2 pad 1: /resistor_network/inputs 16-31/out2_i -> /resistor_network/OUT2
- R24_2 pad 2: /resistor_network/inputs 16-31/in24_v -> /C24
- R24_3 pad 1: /resistor_network/inputs 16-31/out3_i -> /resistor_network/OUT3
- R24_3 pad 2: /resistor_network/inputs 16-31/in24_v -> /C24
- R24_4 pad 1: /resistor_network/inputs 16-31/out4_i -> /resistor_network/OUT4
- R24_4 pad 2: /resistor_network/inputs 16-31/in24_v -> /C24
- R24_5 pad 1: /resistor_network/inputs 16-31/out5_i -> /resistor_network/OUT5
- R24_5 pad 2: /resistor_network/inputs 16-31/in24_v -> /C24
- R24_6 pad 1: /resistor_network/inputs 16-31/out6_i -> /resistor_network/OUT6
- R24_6 pad 2: /resistor_network/inputs 16-31/in24_v -> /C24
- R24_7 pad 1: /resistor_network/inputs 16-31/out7_i -> /resistor_network/OUT7
- R24_7 pad 2: /resistor_network/inputs 16-31/in24_v -> /C24
- R24_8 pad 1: /resistor_network/inputs 16-31/out8_i -> /resistor_network/OUT8
- R24_8 pad 2: /resistor_network/inputs 16-31/in24_v -> /C24
- R24_9 pad 1: /resistor_network/inputs 16-31/out9_i -> /resistor_network/OUT9
- R24_9 pad 2: /resistor_network/inputs 16-31/in24_v -> /C24
- R25_0 pad 1: /resistor_network/inputs 16-31/out0_i -> /resistor_network/OUT0
- R25_0 pad 2: /resistor_network/inputs 16-31/in25_v -> /C25
- R25_1 pad 1: /resistor_network/inputs 16-31/out1_i -> /resistor_network/OUT1
- R25_1 pad 2: /resistor_network/inputs 16-31/in25_v -> /C25
- R25_2 pad 1: /resistor_network/inputs 16-31/out2_i -> /resistor_network/OUT2
- R25_2 pad 2: /resistor_network/inputs 16-31/in25_v -> /C25
- R25_3 pad 1: /resistor_network/inputs 16-31/out3_i -> /resistor_network/OUT3
- R25_3 pad 2: /resistor_network/inputs 16-31/in25_v -> /C25
- R25_4 pad 1: /resistor_network/inputs 16-31/out4_i -> /resistor_network/OUT4
- R25_4 pad 2: /resistor_network/inputs 16-31/in25_v -> /C25
- R25_5 pad 1: /resistor_network/inputs 16-31/out5_i -> /resistor_network/OUT5
- R25_5 pad 2: /resistor_network/inputs 16-31/in25_v -> /C25
- R25_6 pad 1: /resistor_network/inputs 16-31/out6_i -> /resistor_network/OUT6
- R25_6 pad 2: /resistor_network/inputs 16-31/in25_v -> /C25
- R25_7 pad 1: /resistor_network/inputs 16-31/out7_i -> /resistor_network/OUT7
- R25_7 pad 2: /resistor_network/inputs 16-31/in25_v -> /C25
- R25_8 pad 1: /resistor_network/inputs 16-31/out8_i -> /resistor_network/OUT8
- R25_8 pad 2: /resistor_network/inputs 16-31/in25_v -> /C25
- R25_9 pad 1: /resistor_network/inputs 16-31/out9_i -> /resistor_network/OUT9
- R25_9 pad 2: /resistor_network/inputs 16-31/in25_v -> /C25
- R26_0 pad 1: /resistor_network/inputs 16-31/out0_i -> /resistor_network/OUT0
- R26_0 pad 2: /resistor_network/inputs 16-31/in26_v -> /C26
- R26_1 pad 1: /resistor_network/inputs 16-31/out1_i -> /resistor_network/OUT1
- R26_1 pad 2: /resistor_network/inputs 16-31/in26_v -> /C26
- R26_2 pad 1: /resistor_network/inputs 16-31/out2_i -> /resistor_network/OUT2
- R26_2 pad 2: /resistor_network/inputs 16-31/in26_v -> /C26
- R26_3 pad 1: /resistor_network/inputs 16-31/out3_i -> /resistor_network/OUT3
- R26_3 pad 2: /resistor_network/inputs 16-31/in26_v -> /C26
- R26_4 pad 1: /resistor_network/inputs 16-31/out4_i -> /resistor_network/OUT4
- R26_4 pad 2: /resistor_network/inputs 16-31/in26_v -> /C26
- R26_5 pad 1: /resistor_network/inputs 16-31/out5_i -> /resistor_network/OUT5
- R26_5 pad 2: /resistor_network/inputs 16-31/in26_v -> /C26
- R26_6 pad 1: /resistor_network/inputs 16-31/out6_i -> /resistor_network/OUT6
- R26_6 pad 2: /resistor_network/inputs 16-31/in26_v -> /C26
- R26_7 pad 1: /resistor_network/inputs 16-31/out7_i -> /resistor_network/OUT7
- R26_7 pad 2: /resistor_network/inputs 16-31/in26_v -> /C26
- R26_8 pad 1: /resistor_network/inputs 16-31/out8_i -> /resistor_network/OUT8
- R26_8 pad 2: /resistor_network/inputs 16-31/in26_v -> /C26
- R26_9 pad 1: /resistor_network/inputs 16-31/out9_i -> /resistor_network/OUT9
- R26_9 pad 2: /resistor_network/inputs 16-31/in26_v -> /C26
- R27_0 pad 1: /resistor_network/inputs 16-31/out0_i -> /resistor_network/OUT0
- R27_0 pad 2: /resistor_network/inputs 16-31/in27_v -> /C27
- R27_1 pad 1: /resistor_network/inputs 16-31/out1_i -> /resistor_network/OUT1
- R27_1 pad 2: /resistor_network/inputs 16-31/in27_v -> /C27
- R27_2 pad 1: /resistor_network/inputs 16-31/out2_i -> /resistor_network/OUT2
- R27_2 pad 2: /resistor_network/inputs 16-31/in27_v -> /C27
- R27_3 pad 1: /resistor_network/inputs 16-31/out3_i -> /resistor_network/OUT3
- R27_3 pad 2: /resistor_network/inputs 16-31/in27_v -> /C27
- R27_4 pad 1: /resistor_network/inputs 16-31/out4_i -> /resistor_network/OUT4
- R27_4 pad 2: /resistor_network/inputs 16-31/in27_v -> /C27
- R27_5 pad 1: /resistor_network/inputs 16-31/out5_i -> /resistor_network/OUT5
- R27_5 pad 2: /resistor_network/inputs 16-31/in27_v -> /C27
- R27_6 pad 1: /resistor_network/inputs 16-31/out6_i -> /resistor_network/OUT6
- R27_6 pad 2: /resistor_network/inputs 16-31/in27_v -> /C27
- R27_7 pad 1: /resistor_network/inputs 16-31/out7_i -> /resistor_network/OUT7
- R27_7 pad 2: /resistor_network/inputs 16-31/in27_v -> /C27
- R27_8 pad 1: /resistor_network/inputs 16-31/out8_i -> /resistor_network/OUT8
- R27_8 pad 2: /resistor_network/inputs 16-31/in27_v -> /C27
- R27_9 pad 1: /resistor_network/inputs 16-31/out9_i -> /resistor_network/OUT9
- R27_9 pad 2: /resistor_network/inputs 16-31/in27_v -> /C27
- R28_0 pad 1: /resistor_network/inputs 16-31/out0_i -> /resistor_network/OUT0
- R28_0 pad 2: /resistor_network/inputs 16-31/in28_v -> /C28
- R28_1 pad 1: /resistor_network/inputs 16-31/out1_i -> /resistor_network/OUT1
- R28_1 pad 2: /resistor_network/inputs 16-31/in28_v -> /C28
- R28_2 pad 1: /resistor_network/inputs 16-31/out2_i -> /resistor_network/OUT2
- R28_2 pad 2: /resistor_network/inputs 16-31/in28_v -> /C28
- R28_3 pad 1: /resistor_network/inputs 16-31/out3_i -> /resistor_network/OUT3
- R28_3 pad 2: /resistor_network/inputs 16-31/in28_v -> /C28
- R28_4 pad 1: /resistor_network/inputs 16-31/out4_i -> /resistor_network/OUT4
- R28_4 pad 2: /resistor_network/inputs 16-31/in28_v -> /C28
- R28_5 pad 1: /resistor_network/inputs 16-31/out5_i -> /resistor_network/OUT5
- R28_5 pad 2: /resistor_network/inputs 16-31/in28_v -> /C28
- R28_6 pad 1: /resistor_network/inputs 16-31/out6_i -> /resistor_network/OUT6
- R28_6 pad 2: /resistor_network/inputs 16-31/in28_v -> /C28
- R28_7 pad 1: /resistor_network/inputs 16-31/out7_i -> /resistor_network/OUT7
- R28_7 pad 2: /resistor_network/inputs 16-31/in28_v -> /C28
- R28_8 pad 1: /resistor_network/inputs 16-31/out8_i -> /resistor_network/OUT8
- R28_8 pad 2: /resistor_network/inputs 16-31/in28_v -> /C28
- R28_9 pad 1: /resistor_network/inputs 16-31/out9_i -> /resistor_network/OUT9
- R28_9 pad 2: /resistor_network/inputs 16-31/in28_v -> /C28
- R29_0 pad 1: /resistor_network/inputs 16-31/out0_i -> /resistor_network/OUT0
- R29_0 pad 2: /resistor_network/inputs 16-31/in29_v -> /C29
- R29_1 pad 1: /resistor_network/inputs 16-31/out1_i -> /resistor_network/OUT1
- R29_1 pad 2: /resistor_network/inputs 16-31/in29_v -> /C29
- R29_2 pad 1: /resistor_network/inputs 16-31/out2_i -> /resistor_network/OUT2
- R29_2 pad 2: /resistor_network/inputs 16-31/in29_v -> /C29
- R29_3 pad 1: /resistor_network/inputs 16-31/out3_i -> /resistor_network/OUT3
- R29_3 pad 2: /resistor_network/inputs 16-31/in29_v -> /C29
- R29_4 pad 1: /resistor_network/inputs 16-31/out4_i -> /resistor_network/OUT4
- R29_4 pad 2: /resistor_network/inputs 16-31/in29_v -> /C29
- R29_5 pad 1: /resistor_network/inputs 16-31/out5_i -> /resistor_network/OUT5
- R29_5 pad 2: /resistor_network/inputs 16-31/in29_v -> /C29
- R29_6 pad 1: /resistor_network/inputs 16-31/out6_i -> /resistor_network/OUT6
- R29_6 pad 2: /resistor_network/inputs 16-31/in29_v -> /C29
- R29_7 pad 1: /resistor_network/inputs 16-31/out7_i -> /resistor_network/OUT7
- R29_7 pad 2: /resistor_network/inputs 16-31/in29_v -> /C29
- R29_8 pad 1: /resistor_network/inputs 16-31/out8_i -> /resistor_network/OUT8
- R29_8 pad 2: /resistor_network/inputs 16-31/in29_v -> /C29
- R29_9 pad 1: /resistor_network/inputs 16-31/out9_i -> /resistor_network/OUT9
- R29_9 pad 2: /resistor_network/inputs 16-31/in29_v -> /C29
- R3 pad 1: /op_amps/out3_v -> Net-(R3-Pad1)
- R30_0 pad 1: /resistor_network/inputs 16-31/out0_i -> /resistor_network/OUT0
- R30_0 pad 2: /resistor_network/inputs 16-31/in30_v -> /C30
- R30_1 pad 1: /resistor_network/inputs 16-31/out1_i -> /resistor_network/OUT1
- R30_1 pad 2: /resistor_network/inputs 16-31/in30_v -> /C30
- R30_2 pad 1: /resistor_network/inputs 16-31/out2_i -> /resistor_network/OUT2
- R30_2 pad 2: /resistor_network/inputs 16-31/in30_v -> /C30
- R30_3 pad 1: /resistor_network/inputs 16-31/out3_i -> /resistor_network/OUT3
- R30_3 pad 2: /resistor_network/inputs 16-31/in30_v -> /C30
- R30_4 pad 1: /resistor_network/inputs 16-31/out4_i -> /resistor_network/OUT4
- R30_4 pad 2: /resistor_network/inputs 16-31/in30_v -> /C30
- R30_5 pad 1: /resistor_network/inputs 16-31/out5_i -> /resistor_network/OUT5
- R30_5 pad 2: /resistor_network/inputs 16-31/in30_v -> /C30
- R30_6 pad 1: /resistor_network/inputs 16-31/out6_i -> /resistor_network/OUT6
- R30_6 pad 2: /resistor_network/inputs 16-31/in30_v -> /C30
- R30_7 pad 1: /resistor_network/inputs 16-31/out7_i -> /resistor_network/OUT7
- R30_7 pad 2: /resistor_network/inputs 16-31/in30_v -> /C30
- R30_8 pad 1: /resistor_network/inputs 16-31/out8_i -> /resistor_network/OUT8
- R30_8 pad 2: /resistor_network/inputs 16-31/in30_v -> /C30
- R30_9 pad 1: /resistor_network/inputs 16-31/out9_i -> /resistor_network/OUT9
- R30_9 pad 2: /resistor_network/inputs 16-31/in30_v -> /C30
- R31_0 pad 1: /resistor_network/inputs 16-31/out0_i -> /resistor_network/OUT0
- R31_0 pad 2: /resistor_network/inputs 16-31/in31_v -> /C31
- R31_1 pad 1: /resistor_network/inputs 16-31/out1_i -> /resistor_network/OUT1
- R31_1 pad 2: /resistor_network/inputs 16-31/in31_v -> /C31
- R31_2 pad 1: /resistor_network/inputs 16-31/out2_i -> /resistor_network/OUT2
- R31_2 pad 2: /resistor_network/inputs 16-31/in31_v -> /C31
- R31_3 pad 1: /resistor_network/inputs 16-31/out3_i -> /resistor_network/OUT3
- R31_3 pad 2: /resistor_network/inputs 16-31/in31_v -> /C31
- R31_4 pad 1: /resistor_network/inputs 16-31/out4_i -> /resistor_network/OUT4
- R31_4 pad 2: /resistor_network/inputs 16-31/in31_v -> /C31
- R31_5 pad 1: /resistor_network/inputs 16-31/out5_i -> /resistor_network/OUT5
- R31_5 pad 2: /resistor_network/inputs 16-31/in31_v -> /C31
- R31_6 pad 1: /resistor_network/inputs 16-31/out6_i -> /resistor_network/OUT6
- R31_6 pad 2: /resistor_network/inputs 16-31/in31_v -> /C31
- R31_7 pad 1: /resistor_network/inputs 16-31/out7_i -> /resistor_network/OUT7
- R31_7 pad 2: /resistor_network/inputs 16-31/in31_v -> /C31
- R31_8 pad 1: /resistor_network/inputs 16-31/out8_i -> /resistor_network/OUT8
- R31_8 pad 2: /resistor_network/inputs 16-31/in31_v -> /C31
- R31_9 pad 1: /resistor_network/inputs 16-31/out9_i -> /resistor_network/OUT9
- R31_9 pad 2: /resistor_network/inputs 16-31/in31_v -> /C31
- R32_0 pad 1: /resistor_network/inputs 32-47/out0_i -> /resistor_network/OUT0
- R32_0 pad 2: /resistor_network/inputs 32-47/in32_v -> /C32
- R32_1 pad 1: /resistor_network/inputs 32-47/out1_i -> /resistor_network/OUT1
- R32_1 pad 2: /resistor_network/inputs 32-47/in32_v -> /C32
- R32_2 pad 1: /resistor_network/inputs 32-47/out2_i -> /resistor_network/OUT2
- R32_2 pad 2: /resistor_network/inputs 32-47/in32_v -> /C32
- R32_3 pad 1: /resistor_network/inputs 32-47/out3_i -> /resistor_network/OUT3
- R32_3 pad 2: /resistor_network/inputs 32-47/in32_v -> /C32
- R32_4 pad 1: /resistor_network/inputs 32-47/out4_i -> /resistor_network/OUT4
- R32_4 pad 2: /resistor_network/inputs 32-47/in32_v -> /C32
- R32_5 pad 1: /resistor_network/inputs 32-47/out5_i -> /resistor_network/OUT5
- R32_5 pad 2: /resistor_network/inputs 32-47/in32_v -> /C32
- R32_6 pad 1: /resistor_network/inputs 32-47/out6_i -> /resistor_network/OUT6
- R32_6 pad 2: /resistor_network/inputs 32-47/in32_v -> /C32
- R32_7 pad 1: /resistor_network/inputs 32-47/out7_i -> /resistor_network/OUT7
- R32_7 pad 2: /resistor_network/inputs 32-47/in32_v -> /C32
- R32_8 pad 1: /resistor_network/inputs 32-47/out8_i -> /resistor_network/OUT8
- R32_8 pad 2: /resistor_network/inputs 32-47/in32_v -> /C32
- R32_9 pad 1: /resistor_network/inputs 32-47/out9_i -> /resistor_network/OUT9
- R32_9 pad 2: /resistor_network/inputs 32-47/in32_v -> /C32
- R33_0 pad 1: /resistor_network/inputs 32-47/out0_i -> /resistor_network/OUT0
- R33_0 pad 2: /resistor_network/inputs 32-47/in33_v -> /C33
- R33_1 pad 1: /resistor_network/inputs 32-47/out1_i -> /resistor_network/OUT1
- R33_1 pad 2: /resistor_network/inputs 32-47/in33_v -> /C33
- R33_2 pad 1: /resistor_network/inputs 32-47/out2_i -> /resistor_network/OUT2
- R33_2 pad 2: /resistor_network/inputs 32-47/in33_v -> /C33
- R33_3 pad 1: /resistor_network/inputs 32-47/out3_i -> /resistor_network/OUT3
- R33_3 pad 2: /resistor_network/inputs 32-47/in33_v -> /C33
- R33_4 pad 1: /resistor_network/inputs 32-47/out4_i -> /resistor_network/OUT4
- R33_4 pad 2: /resistor_network/inputs 32-47/in33_v -> /C33
- R33_5 pad 1: /resistor_network/inputs 32-47/out5_i -> /resistor_network/OUT5
- R33_5 pad 2: /resistor_network/inputs 32-47/in33_v -> /C33
- R33_6 pad 1: /resistor_network/inputs 32-47/out6_i -> /resistor_network/OUT6
- R33_6 pad 2: /resistor_network/inputs 32-47/in33_v -> /C33
- R33_7 pad 1: /resistor_network/inputs 32-47/out7_i -> /resistor_network/OUT7
- R33_7 pad 2: /resistor_network/inputs 32-47/in33_v -> /C33
- R33_8 pad 1: /resistor_network/inputs 32-47/out8_i -> /resistor_network/OUT8
- R33_8 pad 2: /resistor_network/inputs 32-47/in33_v -> /C33
- R33_9 pad 1: /resistor_network/inputs 32-47/out9_i -> /resistor_network/OUT9
- R33_9 pad 2: /resistor_network/inputs 32-47/in33_v -> /C33
- R34_0 pad 1: /resistor_network/inputs 32-47/out0_i -> /resistor_network/OUT0
- R34_0 pad 2: /resistor_network/inputs 32-47/in34_v -> /C34
- R34_1 pad 1: /resistor_network/inputs 32-47/out1_i -> /resistor_network/OUT1
- R34_1 pad 2: /resistor_network/inputs 32-47/in34_v -> /C34
- R34_2 pad 1: /resistor_network/inputs 32-47/out2_i -> /resistor_network/OUT2
- R34_2 pad 2: /resistor_network/inputs 32-47/in34_v -> /C34
- R34_3 pad 1: /resistor_network/inputs 32-47/out3_i -> /resistor_network/OUT3
- R34_3 pad 2: /resistor_network/inputs 32-47/in34_v -> /C34
- R34_4 pad 1: /resistor_network/inputs 32-47/out4_i -> /resistor_network/OUT4
- R34_4 pad 2: /resistor_network/inputs 32-47/in34_v -> /C34
- R34_5 pad 1: /resistor_network/inputs 32-47/out5_i -> /resistor_network/OUT5
- R34_5 pad 2: /resistor_network/inputs 32-47/in34_v -> /C34
- R34_6 pad 1: /resistor_network/inputs 32-47/out6_i -> /resistor_network/OUT6
- R34_6 pad 2: /resistor_network/inputs 32-47/in34_v -> /C34
- R34_7 pad 1: /resistor_network/inputs 32-47/out7_i -> /resistor_network/OUT7
- R34_7 pad 2: /resistor_network/inputs 32-47/in34_v -> /C34
- R34_8 pad 1: /resistor_network/inputs 32-47/out8_i -> /resistor_network/OUT8
- R34_8 pad 2: /resistor_network/inputs 32-47/in34_v -> /C34
- R34_9 pad 1: /resistor_network/inputs 32-47/out9_i -> /resistor_network/OUT9
- R34_9 pad 2: /resistor_network/inputs 32-47/in34_v -> /C34
- R35_0 pad 1: /resistor_network/inputs 32-47/out0_i -> /resistor_network/OUT0
- R35_0 pad 2: /resistor_network/inputs 32-47/in35_v -> /C35
- R35_1 pad 1: /resistor_network/inputs 32-47/out1_i -> /resistor_network/OUT1
- R35_1 pad 2: /resistor_network/inputs 32-47/in35_v -> /C35
- R35_2 pad 1: /resistor_network/inputs 32-47/out2_i -> /resistor_network/OUT2
- R35_2 pad 2: /resistor_network/inputs 32-47/in35_v -> /C35
- R35_3 pad 1: /resistor_network/inputs 32-47/out3_i -> /resistor_network/OUT3
- R35_3 pad 2: /resistor_network/inputs 32-47/in35_v -> /C35
- R35_4 pad 1: /resistor_network/inputs 32-47/out4_i -> /resistor_network/OUT4
- R35_4 pad 2: /resistor_network/inputs 32-47/in35_v -> /C35
- R35_5 pad 1: /resistor_network/inputs 32-47/out5_i -> /resistor_network/OUT5
- R35_5 pad 2: /resistor_network/inputs 32-47/in35_v -> /C35
- R35_6 pad 1: /resistor_network/inputs 32-47/out6_i -> /resistor_network/OUT6
- R35_6 pad 2: /resistor_network/inputs 32-47/in35_v -> /C35
- R35_7 pad 1: /resistor_network/inputs 32-47/out7_i -> /resistor_network/OUT7
- R35_7 pad 2: /resistor_network/inputs 32-47/in35_v -> /C35
- R35_8 pad 1: /resistor_network/inputs 32-47/out8_i -> /resistor_network/OUT8
- R35_8 pad 2: /resistor_network/inputs 32-47/in35_v -> /C35
- R35_9 pad 1: /resistor_network/inputs 32-47/out9_i -> /resistor_network/OUT9
- R35_9 pad 2: /resistor_network/inputs 32-47/in35_v -> /C35
- R36_0 pad 1: /resistor_network/inputs 32-47/out0_i -> /resistor_network/OUT0
- R36_0 pad 2: /resistor_network/inputs 32-47/in36_v -> /C36
- R36_1 pad 1: /resistor_network/inputs 32-47/out1_i -> /resistor_network/OUT1
- R36_1 pad 2: /resistor_network/inputs 32-47/in36_v -> /C36
- R36_2 pad 1: /resistor_network/inputs 32-47/out2_i -> /resistor_network/OUT2
- R36_2 pad 2: /resistor_network/inputs 32-47/in36_v -> /C36
- R36_3 pad 1: /resistor_network/inputs 32-47/out3_i -> /resistor_network/OUT3
- R36_3 pad 2: /resistor_network/inputs 32-47/in36_v -> /C36
- R36_4 pad 1: /resistor_network/inputs 32-47/out4_i -> /resistor_network/OUT4
- R36_4 pad 2: /resistor_network/inputs 32-47/in36_v -> /C36
- R36_5 pad 1: /resistor_network/inputs 32-47/out5_i -> /resistor_network/OUT5
- R36_5 pad 2: /resistor_network/inputs 32-47/in36_v -> /C36
- R36_6 pad 1: /resistor_network/inputs 32-47/out6_i -> /resistor_network/OUT6
- R36_6 pad 2: /resistor_network/inputs 32-47/in36_v -> /C36
- R36_7 pad 1: /resistor_network/inputs 32-47/out7_i -> /resistor_network/OUT7
- R36_7 pad 2: /resistor_network/inputs 32-47/in36_v -> /C36
- R36_8 pad 1: /resistor_network/inputs 32-47/out8_i -> /resistor_network/OUT8
- R36_8 pad 2: /resistor_network/inputs 32-47/in36_v -> /C36
- R36_9 pad 1: /resistor_network/inputs 32-47/out9_i -> /resistor_network/OUT9
- R36_9 pad 2: /resistor_network/inputs 32-47/in36_v -> /C36
- R37_0 pad 1: /resistor_network/inputs 32-47/out0_i -> /resistor_network/OUT0
- R37_0 pad 2: /resistor_network/inputs 32-47/in37_v -> /C37
- R37_1 pad 1: /resistor_network/inputs 32-47/out1_i -> /resistor_network/OUT1
- R37_1 pad 2: /resistor_network/inputs 32-47/in37_v -> /C37
- R37_2 pad 1: /resistor_network/inputs 32-47/out2_i -> /resistor_network/OUT2
- R37_2 pad 2: /resistor_network/inputs 32-47/in37_v -> /C37
- R37_3 pad 1: /resistor_network/inputs 32-47/out3_i -> /resistor_network/OUT3
- R37_3 pad 2: /resistor_network/inputs 32-47/in37_v -> /C37
- R37_4 pad 1: /resistor_network/inputs 32-47/out4_i -> /resistor_network/OUT4
- R37_4 pad 2: /resistor_network/inputs 32-47/in37_v -> /C37
- R37_5 pad 1: /resistor_network/inputs 32-47/out5_i -> /resistor_network/OUT5
- R37_5 pad 2: /resistor_network/inputs 32-47/in37_v -> /C37
- R37_6 pad 1: /resistor_network/inputs 32-47/out6_i -> /resistor_network/OUT6
- R37_6 pad 2: /resistor_network/inputs 32-47/in37_v -> /C37
- R37_7 pad 1: /resistor_network/inputs 32-47/out7_i -> /resistor_network/OUT7
- R37_7 pad 2: /resistor_network/inputs 32-47/in37_v -> /C37
- R37_8 pad 1: /resistor_network/inputs 32-47/out8_i -> /resistor_network/OUT8
- R37_8 pad 2: /resistor_network/inputs 32-47/in37_v -> /C37
- R37_9 pad 1: /resistor_network/inputs 32-47/out9_i -> /resistor_network/OUT9
- R37_9 pad 2: /resistor_network/inputs 32-47/in37_v -> /C37
- R38_0 pad 1: /resistor_network/inputs 32-47/out0_i -> /resistor_network/OUT0
- R38_0 pad 2: /resistor_network/inputs 32-47/in38_v -> /C38
- R38_1 pad 1: /resistor_network/inputs 32-47/out1_i -> /resistor_network/OUT1
- R38_1 pad 2: /resistor_network/inputs 32-47/in38_v -> /C38
- R38_2 pad 1: /resistor_network/inputs 32-47/out2_i -> /resistor_network/OUT2
- R38_2 pad 2: /resistor_network/inputs 32-47/in38_v -> /C38
- R38_3 pad 1: /resistor_network/inputs 32-47/out3_i -> /resistor_network/OUT3
- R38_3 pad 2: /resistor_network/inputs 32-47/in38_v -> /C38
- R38_4 pad 1: /resistor_network/inputs 32-47/out4_i -> /resistor_network/OUT4
- R38_4 pad 2: /resistor_network/inputs 32-47/in38_v -> /C38
- R38_5 pad 1: /resistor_network/inputs 32-47/out5_i -> /resistor_network/OUT5
- R38_5 pad 2: /resistor_network/inputs 32-47/in38_v -> /C38
- R38_6 pad 1: /resistor_network/inputs 32-47/out6_i -> /resistor_network/OUT6
- R38_6 pad 2: /resistor_network/inputs 32-47/in38_v -> /C38
- R38_7 pad 1: /resistor_network/inputs 32-47/out7_i -> /resistor_network/OUT7
- R38_7 pad 2: /resistor_network/inputs 32-47/in38_v -> /C38
- R38_8 pad 1: /resistor_network/inputs 32-47/out8_i -> /resistor_network/OUT8
- R38_8 pad 2: /resistor_network/inputs 32-47/in38_v -> /C38
- R38_9 pad 1: /resistor_network/inputs 32-47/out9_i -> /resistor_network/OUT9
- R38_9 pad 2: /resistor_network/inputs 32-47/in38_v -> /C38
- R39_0 pad 1: /resistor_network/inputs 32-47/out0_i -> /resistor_network/OUT0
- R39_0 pad 2: /resistor_network/inputs 32-47/in39_v -> /C39
- R39_1 pad 1: /resistor_network/inputs 32-47/out1_i -> /resistor_network/OUT1
- R39_1 pad 2: /resistor_network/inputs 32-47/in39_v -> /C39
- R39_2 pad 1: /resistor_network/inputs 32-47/out2_i -> /resistor_network/OUT2
- R39_2 pad 2: /resistor_network/inputs 32-47/in39_v -> /C39
- R39_3 pad 1: /resistor_network/inputs 32-47/out3_i -> /resistor_network/OUT3
- R39_3 pad 2: /resistor_network/inputs 32-47/in39_v -> /C39
- R39_4 pad 1: /resistor_network/inputs 32-47/out4_i -> /resistor_network/OUT4
- R39_4 pad 2: /resistor_network/inputs 32-47/in39_v -> /C39
- R39_5 pad 1: /resistor_network/inputs 32-47/out5_i -> /resistor_network/OUT5
- R39_5 pad 2: /resistor_network/inputs 32-47/in39_v -> /C39
- R39_6 pad 1: /resistor_network/inputs 32-47/out6_i -> /resistor_network/OUT6
- R39_6 pad 2: /resistor_network/inputs 32-47/in39_v -> /C39
- R39_7 pad 1: /resistor_network/inputs 32-47/out7_i -> /resistor_network/OUT7
- R39_7 pad 2: /resistor_network/inputs 32-47/in39_v -> /C39
- R39_8 pad 1: /resistor_network/inputs 32-47/out8_i -> /resistor_network/OUT8
- R39_8 pad 2: /resistor_network/inputs 32-47/in39_v -> /C39
- R39_9 pad 1: /resistor_network/inputs 32-47/out9_i -> /resistor_network/OUT9
- R39_9 pad 2: /resistor_network/inputs 32-47/in39_v -> /C39
- R4 pad 1: /op_amps/out4_v -> Net-(R4-Pad1)
- R40_0 pad 1: /resistor_network/inputs 32-47/out0_i -> /resistor_network/OUT0
- R40_0 pad 2: /resistor_network/inputs 32-47/in40_v -> /C40
- R40_1 pad 1: /resistor_network/inputs 32-47/out1_i -> /resistor_network/OUT1
- R40_1 pad 2: /resistor_network/inputs 32-47/in40_v -> /C40
- R40_2 pad 1: /resistor_network/inputs 32-47/out2_i -> /resistor_network/OUT2
- R40_2 pad 2: /resistor_network/inputs 32-47/in40_v -> /C40
- R40_3 pad 1: /resistor_network/inputs 32-47/out3_i -> /resistor_network/OUT3
- R40_3 pad 2: /resistor_network/inputs 32-47/in40_v -> /C40
- R40_4 pad 1: /resistor_network/inputs 32-47/out4_i -> /resistor_network/OUT4
- R40_4 pad 2: /resistor_network/inputs 32-47/in40_v -> /C40
- R40_5 pad 1: /resistor_network/inputs 32-47/out5_i -> /resistor_network/OUT5
- R40_5 pad 2: /resistor_network/inputs 32-47/in40_v -> /C40
- R40_6 pad 1: /resistor_network/inputs 32-47/out6_i -> /resistor_network/OUT6
- R40_6 pad 2: /resistor_network/inputs 32-47/in40_v -> /C40
- R40_7 pad 1: /resistor_network/inputs 32-47/out7_i -> /resistor_network/OUT7
- R40_7 pad 2: /resistor_network/inputs 32-47/in40_v -> /C40
- R40_8 pad 1: /resistor_network/inputs 32-47/out8_i -> /resistor_network/OUT8
- R40_8 pad 2: /resistor_network/inputs 32-47/in40_v -> /C40
- R40_9 pad 1: /resistor_network/inputs 32-47/out9_i -> /resistor_network/OUT9
- R40_9 pad 2: /resistor_network/inputs 32-47/in40_v -> /C40
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Routing:
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Other:
- board outline added: 262.9 x 181.6 mm

Commit message: Commit before Auto-Routing
Because this tool *might* just fuck everything up, so I want a "shit go back" point
Parts:
- moved R90 76.9 mm to (106.7, 171.4)
- moved R91 74.4 mm to (106.7, 166.4)
- moved R80 68.1 mm to (106.7, 148.6)
- moved R81 67.0 mm to (106.7, 143.5)
- moved R8 66.3 mm to (106.7, 153.7)
- moved R70 62.3 mm to (80.0, 180.3)
- moved R5 59.7 mm to (80.0, 144.8)
- moved R71 58.4 mm to (80.0, 175.3)
- moved U2 55.1 mm to (38.1, 180.3)
- moved R20 49.6 mm to (29.2, 180.3)
- moved R02 49.5 mm to (29.2, 134.6)
- moved U3 49.5 mm to (63.5, 148.6)
- moved R60 47.6 mm to (80.0, 158.8)
- moved U5 46.6 mm to (88.9, 139.7)
- moved R61 44.9 mm to (80.0, 153.7)
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Routing:
- net /C4: track 0.00 -> 70.6 mm, vias 0 -> 10
- net /C9: track 0.00 -> 69.3 mm, vias 0 -> 10
- net /C7: track 0.00 -> 69.3 mm, vias 0 -> 10
- net /C63: track 0.00 -> 69.3 mm, vias 0 -> 10
- net /C62: track 0.00 -> 69.3 mm, vias 0 -> 10
- net /C61: track 0.00 -> 69.3 mm, vias 0 -> 10
- net /C59: track 0.00 -> 69.3 mm, vias 0 -> 10
- net /C57: track 0.00 -> 69.3 mm, vias 0 -> 10
- net /C55: track 0.00 -> 69.3 mm, vias 0 -> 10
- net /C53: track 0.00 -> 69.3 mm, vias 0 -> 10
- net /C51: track 0.00 -> 69.3 mm, vias 0 -> 10
- net /C49: track 0.00 -> 69.3 mm, vias 0 -> 10
- net /C47: track 0.00 -> 69.3 mm, vias 0 -> 10
- net /C46: track 0.00 -> 69.3 mm, vias 0 -> 10
- net /C45: track 0.00 -> 69.3 mm, vias 0 -> 10
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
Commit message: Commit post-autoroute
Something weird happened in github so I think this should be the same commit
Routing:
- net VDD: track 0.00 -> 349.5 mm, vias 0 -> 4
- net GND: track 0.00 -> 322.7 mm, vias 0 -> 5
- net /C63: track 69.3 -> 347.9 mm, vias 10 -> 11
- net /C62: track 69.3 -> 338.8 mm, vias 10 -> 11
- net /C61: track 69.3 -> 336.4 mm, vias 10 -> 11
- net /C22: track 69.3 -> 333.1 mm
- net /C60: track 69.3 -> 320.0 mm, vias 10 -> 12
- net /C47: track 69.3 -> 317.2 mm
- net /C46: track 69.3 -> 315.9 mm
- net /C23: track 82.0 -> 327.8 mm
- net /C59: track 69.3 -> 314.4 mm, vias 10 -> 11
- net /C20: track 69.3 -> 312.2 mm
- net /resistor_network/OUT0: track 727.6 -> 967.4 mm, vias 0 -> 3
- net /C58: track 69.3 -> 303.2 mm, vias 10 -> 12
- net /C57: track 69.3 -> 303.0 mm, vias 10 -> 11
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
Commit message: Post Auto-Route Commit
Deleted all the traces, then let the autorouter do its thing. It worked really well actually, so we'll probably just keep this.
Routing:
- net /resistor_network/OUT8: track 857.6 -> 1006.0 mm, vias 4 -> 5
- net /resistor_network/OUT1: track 946.9 -> 1093.6 mm, vias 3 -> 6
- net /resistor_network/OUT2: track 944.4 -> 1083.6 mm, vias 5 -> 6
- net /resistor_network/OUT0: track 967.4 -> 833.1 mm, vias 3 -> 6
- net /resistor_network/OUT9: track 858.2 -> 772.6 mm, vias 3 -> 0
- net /C40: track 269.7 -> 326.1 mm, vias 10 -> 5
- net /C37: track 233.7 -> 288.4 mm, vias 10 -> 2
- net /resistor_network/OUT3: track 923.4 -> 872.1 mm, vias 4 -> 6
- net /C22: track 333.1 -> 378.3 mm, vias 10 -> 0
- net /C46: track 315.9 -> 358.7 mm, vias 10 -> 0
- net /C58: track 303.2 -> 342.8 mm, vias 12 -> 4
- net /C62: track 338.8 -> 374.5 mm, vias 11 -> 1
- net /resistor_network/OUT6: track 886.5 -> 852.5 mm, vias 4 -> 5
- net /C61: track 336.4 -> 304.0 mm, vias 11 -> 1
- net /resistor_network/OUT7: track 896.8 -> 928.5 mm, vias 4 -> 8
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
Commit message: Commit with Plane
Added some copper planes to make the etching process go faster
Routing:
- added copper zone on B.Cu, net GND
- added copper zone on F.Cu, net VDD
Changed lines of the file:
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@@
   (segment (start 114.47 170.5) (end 111.5484 170.5) (width 0.25) (layer F.Cu) (net 96))
   (segment (start 107.1807 172.6254) (end 106.0053 171.45) (width 0.25) (layer F.Cu) (net 96))
+  (zone (net 75) (net_name VDD) (layer F.Cu) (hatch edge 0.508)
+    (connect_pads (clearance 0.508))
+    (min_thickness 0.254)
+    (fill yes (arc_segments 16) (thermal_gap 0.508) (thermal_bridge_width 0.508))
+    (polygon
+      (pts
+        (xy 278.13 15.24) (xy 278.13 196.85) (xy 15.24 196.85) (xy 15.24 15.24)
+      )
+    )
+  )
+  (zone (net 76) (net_name GND) (layer B.Cu) (hatch edge 0.508)
+    (connect_pads (clearance 0.508))
+    (min_thickness 0.254)
+    (fill yes (arc_segments 16) (thermal_gap 0.508) (thermal_bridge_width 0.508))
+    (polygon
+      (pts
+        (xy 15.24 15.24) (xy 15.24 196.85) (xy 278.13 196.85) (xy 278.13 15.24)
+      )
+    )
+  )
 )
